File: HARTShield.sch (EAGLE design)
At the start: 31 parts, among them Y1 3M6864

Commit message: Minor fixes on partlist.
Parts:
- AMP1: value OP177GS -> OP37GS; device hartmodems:OP177GS -> hartmodems:OP37GS
Changed lines of the file:
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@@
 <part name="C11" library="SparkFun-Capacitors" deviceset="10UF-TANT" device="" value="10uF"/>
 <part name="SUPPLY12" library="SparkFun-Aesthetics" deviceset="VNEG" device="" value="-5V"/>
-<part name="AMP1" library="hartmodems" deviceset="OP177G" device="S"/>
+<part name="AMP1" library="hartmodems" deviceset="OP37G" device="S"/>
 <part name="SUPPLY10" library="SparkFun-Aesthetics" deviceset="VNEG" device="" value="-5V"/>
 <part name="SUPPLY13" library="SparkFun-Aesthetics" deviceset="5V" device=""/>
